File: slimevr.kicad_pcb (KiCad board)
At the start: 4 copper layers, 40 x 46 mm, 95 parts, among them J101 VBUS DNI, J102 Serial Connector DNI, J103 External Motion, J201 USB_C_Receptacle_USB2.0_GCT, J202 BAT w/THERM, J203 BAT_NO_THERM, J204 BAT w/THERM, Q201 UMH3N, SW101 SW_Push, SW102 SW_Push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

Commit message: Minor cleanup
Signed-off-by: Aaron Williams <aaron.w2@gmail.com>
Parts:
- R109, R110: value 2.2K -> 4.7K
- moved R217 5.05 mm to (108.6, 79.5), turned to 0 degrees
- moved R218 4.80 mm to (135.6, 75.7)
- moved FID101 3.44 mm to (110.9, 82.7)
- moved C209 2.77 mm to (133.5, 79.6), turned to -90 degrees
- moved U206 1.50 mm to (135.7, 79.6)
- moved C210 1.50 mm to (135.6, 77.2)
- moved C106 0.54 mm to (114.8, 69.9)
- moved J203 0.45 mm to (125.5, 86.2)
- moved Y101 0.32 mm to (114.5, 67.0)
- moved J201 0.21 mm to (117.8, 93.2)
Routing:
- net SHUTDOWN: track 33.0 -> 26.5 mm
- net /USB and  Power/RTS: track 15.9 -> 21.9 mm, vias 2 -> 3
- net /USB and  Power/DTR: track 14.5 -> 18.9 mm
- net /USB and  Power/CC2: track 5.77 -> 9.03 mm
- net /USB and  Power/BATT+: track 32.3 -> 35.1 mm
- net /USB and  Power/USB_CHGEN: track 25.1 -> 22.7 mm, vias 2 -> 3
- net /USB and  Power/THERM: track 12.8 -> 10.5 mm
- net GND: track 29.7 -> 31.6 mm, vias 188 -> 189
- net Net-(R216-Pad1): track 3.56 -> 5.08 mm
- net /USB and  Power/~{PG}: track 17.6 -> 16.4 mm
- net /USB and  Power/TX_LED: track 31.0 -> 30.1 mm
- net /USB and  Power/USB_CHG500MA: track 15.0 -> 14.1 mm
- net /~{RST}: track 6.42 -> 5.66 mm
- net /B_CLK: track 9.53 -> 8.81 mm
- net CHG_EN: track 47.3 -> 48.1 mm
- removed copper zone on In2.Cu, net GND
