File: slimevr.kicad_sch (KiCad schematic)
At the start: 40 parts, among them J101 VBUS DNI, J102 Serial Connector DNI, J103 External Motion, SW101 SW_Push, SW102 SW_Push, U101 BNO085, U102 ESP-WROOM-02, Y101 OM-7604-C7

Commit message: Minor cleanup
Signed-off-by: Aaron Williams <aaron.w2@gmail.com>
Parts:
- R109, R110: value 2.2K -> 4.7K; DESC 0 Ohms Jumper 0.063W, 1/16W Chip Resistor 0402 (1005 Metric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 -> 4.7 kOhms ±1% 0.1W, 1/10W Chip Resistor 0603 (1608 Metric) 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
Other:
- moved on the sheet: C101, C102, FB101
